File: hw/maqueen/maqueen.kicad_sch (KiCad schematic)
At the start: 44 parts, among them IC1 MSP430FR2355TPT, J1 conn_DFrobot, J2 ESP01, J3 SBW, SW1 RST, U1 LMV324, Y1 Crystal

Commit message: canvis def disseny
Parts:
- added C4: 100n, Capacitor_SMD:C_0805_2012Metric, symbol Device:C
- D1: footprint (none) -> LED_THT:LED_D1.8mm_W3.3mm_H2.4mm
Connections:
- net +3.3V: now also C4.1
- net GND: now also S1.D1 (NO_2), C4.2
- net WIFI_UART_RX: now also IC1.30 (P2.0/TB1.1/COMP0.O), J2.6 (Pin_6)
- no-connect marks 29 -> 26
Changed lines of the file:
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@@
   (junction (at 341.63 60.96) (diameter 0) (color 0 0 0 0)
   )
+  (junction (at 238.76 148.59) (diameter 0) (color 0 0 0 0)
+  )
   (junction (at 119.38 245.11) (diameter 0) (color 0 0 0 0)
   )
@@
   )
   (junction (at 39.37 182.88) (diameter 0) (color 0 0 0 0)
+  )
+  (junction (at 251.46 140.97) (diameter 0) (color 0 0 0 0)
   )
   (junction (at 320.04 72.39) (diameter 0) (color 0 0 0 0)
@@
   (no_connect (at 168.91 55.88))
   (no_connect (at 196.85 151.13))
-  (no_connect (at 289.56 69.85))
   (no_connect (at 196.85 156.21))
-  (no_connect (at 196.85 143.51))
   (no_connect (at 146.05 204.47))
   (no_connect (at 123.19 80.01))
@@
   (no_connect (at 226.06 146.05))
   (no_connect (at 67.31 151.13))
-  (no_connect (at 238.76 146.05))
   (no_connect (at 226.06 143.51))
   (no_connect (at 196.85 128.27))
@@
     (stroke (width 0) (type default))
   )
+  (wire (pts (xy 209.55 153.67) (xy 209.55 143.51))
+    (stroke (width 0) (type default))
+  )
   (wire (pts (xy 341.63 109.22) (xy 341.63 116.84))
     (stroke (width 0) (type default))
@@
     (stroke (width 0) (type default))
   )
+  (wire (pts (xy 289.56 69.85) (xy 288.29 69.85))
+    (stroke (width 0) (type default))
+  )
   (wire (pts (xy 97.79 78.74) (xy 99.06 78.74))
     (stroke (width 0) (type default))
@@
     (stroke (width 0) (type default))
   )
+  (wire (pts (xy 251.46 140.97) (xy 238.76 140.97))
+    (stroke (width 0) (type default))
+  )
   (wire (pts (xy 67.31 146.05) (xy 35.56 146.05))
     (stroke (width 0) (type default))
@@
     (stroke (width 0) (type default))
   )
+  (wire (pts (xy 238.76 153.67) (xy 209.55 153.67))
+    (stroke (width 0) (type default))
+  )
   (wire (pts (xy 99.06 78.74) (xy 115.57 78.74))
     (stroke (width 0) (type default))
@@
     (stroke (width 0) (type default))
   )
+  (wire (pts (xy 209.55 143.51) (xy 196.85 143.51))
+    (stroke (width 0) (type default))
+  )
   (wire (pts (xy 308.61 123.19) (xy 308.61 124.46))
     (stroke (width 0) (type default))
@@
     (stroke (width 0) (type default))
   )
+  (wire (pts (xy 238.76 148.59) (xy 238.76 153.67))
+    (stroke (width 0) (type default))
+  )
   (wire (pts (xy 299.72 123.19) (xy 308.61 123.19))
     (stroke (width 0) (type default))
@@
     (stroke (width 0) (type default))
   )
+  (wire (pts (xy 238.76 146.05) (xy 238.76 148.59))
+    (stroke (width 0) (type default))
+  )
   (wire (pts (xy 283.21 82.55) (xy 283.21 91.44))
     (stroke (width 0) (type default))
@@
   )
   (wire (pts (xy 153.67 33.02) (xy 168.91 33.02))
+    (stroke (width 0) (type default))
+  )
+  (wire (pts (xy 288.29 69.85) (xy 288.29 76.2))
     (stroke (width 0) (type default))
   )
@@
     )
   )
-  (symbol (lib_id "power:+3.3V") (at 238.76 140.97 0) (unit 1)
+  (symbol (lib_id "power:+3.3V") (at 251.46 140.97 0) (unit 1)
     (in_bom yes) (on_board yes) (dnp no) (fields_autoplaced)
-    (property "Reference" "#PWR04" (at 238.76 144.78 0)
-      (effects (font (size 1.27 1.27)) hide)
-    )
-    (property "Value" "+3.3V" (at 238.76 135.89 0)
-      (effects (font (size 1.27 1.27)))
-    )
-    (property "Footprint" "" (at 238.76 140.97 0)
-      (effects (font (size 1.27 1.27)) hide)
-    )
-    (property "Datasheet" "" (at 238.76 140.97 0)
+    (property "Reference" "#PWR04" (at 251.46 144.78 0)
+      (effects (font (size 1.27 1.27)) hide)
+    )
+    (property "Value" "+3.3V" (at 251.46 135.89 0)
+      (effects (font (size 1.27 1.27)))
+    )
+    (property "Footprint" "" (at 251.46 140.97 0)
+      (effects (font (size 1.27 1.27)) hide)
+    )
+    (property "Datasheet" "" (at 251.46 140.97 0)
       (effects (font (size 1.27 1.27)) hide)
     )
@@
         (path "/4609337f-777a-4f75-ba6f-056b355c5403"
           (reference "#PWR014") (unit 1)
+        )
+      )
+    )
+  )
+  (symbol (lib_id "power:GND") (at 251.46 148.59 0) (mirror y) (unit 1)
+    (in_bom yes) (on_board yes) (dnp no)
+    (property "Reference" "#PWR033" (at 251.46 154.94 0)
+      (effects (font (size 1.27 1.27)) hide)
+    )
+    (property "Value" "GND" (at 251.46 152.4 0)
+      (effects (font (size 1.27 1.27)))
+    )
+    (property "Footprint" "" (at 251.46 148.59 0)
+      (effects (font (size 1.27 1.27)) hide)
+    )
+    (property "Datasheet" "" (at 251.46 148.59 0)
+      (effects (font (size 1.27 1.27)) hide)
+    )
+    (pin "1")
+    (instances
+      (project "maqueen"
+        (path "/4609337f-777a-4f75-ba6f-056b355c5403"
+          (reference "#PWR033") (unit 1)
         )
       )
@@
     )
   )
+  (symbol (lib_id "power:GND") (at 288.29 76.2 0) (mirror y) (unit 1)
+    (in_bom yes) (on_board yes) (dnp no)
+    (property "Reference" "#PWR034" (at 288.29 82.55 0)
+      (effects (font (size 1.27 1.27)) hide)
+    )
+    (property "Value" "GND" (at 288.29 80.01 0)
+      (effects (font (size 1.27 1.27)))
+    )
+    (property "Footprint" "" (at 288.29 76.2 0)
+      (effects (font (size 1.27 1.27)) hide)
+    )
+    (property "Datasheet" "" (at 288.29 76.2 0)
+      (effects (font (size 1.27 1.27)) hide)
+    )
+    (pin "1")
+    (instances
+      (project "maqueen"
+        (path "/4609337f-777a-4f75-ba6f-056b355c5403"
+          (reference "#PWR034") (unit 1)
+        )
+      )
+    )
+  )
   (symbol (lib_id "Device:C") (at 35.56 156.21 0) (unit 1)
     (in_bom yes) (on_board yes) (dnp no)
@@
       (effects (font (size 1.27 1.27)) (justify right))
     )
-    (property "Footprint" "" (at 101.6 248.92 0)
+    (property "Footprint" "LED_THT:LED_D1.8mm_W3.3mm_H2.4mm" (at 101.6 248.92 0)
       (effects (font (size 1.27 1.27)) hide)
     )
@@
         )
       )
+    )
+  )
+  (symbol (lib_id "Device:C") (at 251.46 144.78 0) (mirror y) (unit 1)
+    (in_bom yes) (on_board yes) (dnp no)
+    (property "Reference" "C4" (at 248.92 143.51 0)
+      (effects (font (size 1.27 1.27)) (justify left))
+    )
+    (property "Value" "100n" (at 248.92 146.05 0)
+      (effects (font (size 1.27 1.27)) (justify left))
+    )
+    (property "Footprint" "Capacitor_SMD:C_0805_2012Metric" (at 250.4948 148.59 0)
+      (effects (font (size 1.27 1.27)) hide)
+    )
+    (property "Datasheet" "~" (at 251.46 144.78 0)
+      (effects (font (size 1.27 1.27)) hide)
+    )
+    (pin "2")
+    (pin "1")
+    (instances
+      (project "maqueen"
+        (path "/4609337f-777a-4f75-ba6f-056b355c5403"
+          (reference "C4") (unit 1)
+        )
+      )

Commit message: placa corregida
Connections:
- net WIFI_UART_RX: no longer IC1.30 (P2.0/TB1.1/COMP0.O), J2.6 (Pin_6)
- new net WIFI_CE: IC1.30 (P2.0/TB1.1/COMP0.O), J2.6 (Pin_6)
Changed lines of the file:
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@@
   (junction (at 341.63 60.96) (diameter 0) (color 0 0 0 0)
-  )
-  (junction (at 238.76 148.59) (diameter 0) (color 0 0 0 0)
   )
   (junction (at 119.38 245.11) (diameter 0) (color 0 0 0 0)
@@
     (stroke (width 0) (type default))
   )
-  (wire (pts (xy 209.55 153.67) (xy 209.55 143.51))
+  (wire (pts (xy 212.09 153.67) (xy 212.09 143.51))
     (stroke (width 0) (type default))
   )
@@
     (stroke (width 0) (type default))
   )
-  (wire (pts (xy 238.76 153.67) (xy 209.55 153.67))
+  (wire (pts (xy 240.03 153.67) (xy 212.09 153.67))
     (stroke (width 0) (type default))
   )
@@
     (stroke (width 0) (type default))
   )
+  (wire (pts (xy 240.03 146.05) (xy 238.76 146.05))
+    (stroke (width 0) (type default))
+  )
   (wire (pts (xy 48.26 128.27) (xy 63.5 128.27))
     (stroke (width 0) (type default))
   )
-  (wire (pts (xy 209.55 143.51) (xy 196.85 143.51))
+  (wire (pts (xy 212.09 143.51) (xy 196.85 143.51))
     (stroke (width 0) (type default))
   )
@@
     (stroke (width 0) (type default))
   )
-  (wire (pts (xy 238.76 148.59) (xy 238.76 153.67))
-    (stroke (width 0) (type default))
-  )
   (wire (pts (xy 299.72 123.19) (xy 308.61 123.19))
     (stroke (width 0) (type default))
@@
     (stroke (width 0) (type default))
   )
-  (wire (pts (xy 238.76 146.05) (xy 238.76 148.59))
+  (wire (pts (xy 240.03 146.05) (xy 240.03 153.67))
     (stroke (width 0) (type default))
   )
@@
   )
   (label "P6.3" (at 133.35 223.52 90) (fields_autoplaced)
+    (effects (font (size 1.27 1.27)) (justify left bottom))
+  )
+  (label "WIFI_CE" (at 207.01 143.51 0) (fields_autoplaced)
     (effects (font (size 1.27 1.27)) (justify left bottom))
   )
@@
   (symbol (lib_id "Connector:TestPoint") (at 223.52 140.97 180) (unit 1)
     (in_bom yes) (on_board yes) (dnp no)
-    (property "Reference" "UART_TX1" (at 222.25 146.05 0)
+    (property "Reference" "UART_TX1" (at 223.52 146.05 0)
       (effects (font (size 1.27 1.27)) (justify left))
     )

Commit message: line track works
Other:
- note added: "CLK"
- note added: "LCD"
- note added: "LDR"
- note added: "ROBOT"
- note added: "WIFI"
- moved on the sheet: C1, C4, C7, C9, J2, J3, R10, R11, R13, R5, R6, R7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
